File: CAD/Eagle/STARduino/starduino.brd (EAGLE design)
At the start: 101.6 x 38.1 mm, 97 parts, among them J1 J30J-9J30, J2 MICRO_SD, J3 J30J-15J30, J4 J30J-31J30, Q2 BSS8402DW, Q3 BSS8402DW, Q4 DMMT5401, Q5 DMG2305UX, U1 SSCMNNN015PA2A3, U10 MC14504BDTG, U11 MAX31725MTA+, U12 TCA9535_RTW_24, U13 BMX055, U15 MC74VHC1GT125, U16 PCA9515A, U17 PCA9306DCT, U2 LT3465/A, U3 LTC3112FE, U4 DS3231MZ+, U5 MT25QL01GBBB8ESF-0AAT, U6 ATSAMD21G18, U7 MIC5319, U8 ADXL375BCCZ

Commit message: STARduino and Datalogger
Parts:
- removed C11: 10pF, resistor:C0603
- removed C12, C18: 47pF, resistor:C0603
- removed C13, C29, C6: 100nF, resistor:C0603
- removed C14: 680pF, resistor:C0603
- removed C15, C28, C3, C4, C42: 1uF, resistor:C0603
- removed C19: 47uF, resistor:C1210
- removed C2: 22uF, resistor:C1206
- removed C30: 2.2uF, resistor:C0603
- removed D4: B0520LW-7-F, CM_diodes:SOD123
- removed J1: J30J-9J30, CM_J30J:ZKN-9-J30
- removed J2: MICRO_SD, NR_connectors:MICROSD_PUSH_PUSH_AMPHENOL
- removed L1: 22uH, AR_passives:VLF504012MT(TDK)
- removed L2: 4.7uH, CM_passives:SRP5030
- removed Q4: DMMT5401, transistor-pnp:SOT-26
- removed Q5: DMG2305UX, transistor-fet:SOT23
- removed R10, R31: 10k, resistor:R0603
- removed R32: 47k, resistor:R0603
- removed R33: 1M, resistor:R0603
- removed R4: 6.2, resistor:R0603
- removed R5, R6: 33k, resistor:R0603
- removed R8: 845k, resistor:R0603
- removed R9: 158k, resistor:R0603
- removed U2: LT3465/A, AR_IC:SOT23-6
- removed U3: LTC3112FE, CM_IC:TSSOP20
- removed U7: MIC5319, CM_IC:SOT23-5L
Connections:
- removed net BIAS_GND: J4.3
- removed net BIAS_V: J4.4
- removed net CAM1_C_N: J4.24
- removed net CAM1_C_P: J4.25
- removed net CAM1_D0_N: J4.18
- removed net CAM1_D0_P: J4.19
- removed net CAM1_D1_N: J4.21
- removed net CAM1_D1_P: J4.22
- removed net CAM_CLK: J4.28
- removed net CAM_GPIO: J4.27
- removed net C_3V3: J4.31
- removed net C_SCL0: J4.29
- removed net C_SDA0: J4.30
- removed net FB_5: C11.2, C14.2, R10.1, R8.2, R9.1, U3.3
- removed net LED_GND: J4.2, R4.2, U2.3
- removed net LED_V: C15.1, J4.1, U2.1
- removed net MA1: J4.5
- removed net MA2: J4.6
- removed net MB1: J4.7
- removed net MB2: J4.8
- removed net N$1: Q4.4, Q5.1, R32.2
- removed net N$11: C14.1, R6.1
- removed net N$12: C11.1, R6.2, U3.2
- removed net N$15: L1.P$2, U2.6
- removed net N$2: Q4.1, Q4.2, Q4.3, R31.2
- removed net N$3: R33.1, U3.19
- removed net N$39: C6.1, L2.P$1, U3.15, U3.16
- removed net N$40: C13.1, L2.P$2, U3.12, U3.13
- removed net N$41: C6.2, U3.17
- removed net N$42: C13.2, U3.14
- removed net N$43: C4.1, D4.C, R33.2, U3.18
- removed net N$48: C18.2, R10.2
- removed net N$9: C29.1, U7.4
- removed net VCC: C2.1, C42.1, J1.1, J1.2, U3.5, U3.6, U3.7
- net +3V3: no longer C30.1, J2.4, U7.5
- net +5V: no longer C18.1, C19.1, D4.A, Q4.6, Q5.2, R8.1, U3.9
- net 5V_S: no longer C28.1, C3.1, L1.P$1, Q4.5, Q5.3, U2.5, U7.1, U7.3
- net EXTERNAL_3V3: no longer J4.15
- net GND: no longer C12.2, C15.2, C19.2, C2.2, C28.2, C29.2, C3.2, C30.2, C4.2, C42.2, J1.3, J1.4, J1.5, J2.6, J2.G1, J2.G2, J2.G3, J4.14, J4.17, J4.20, J4.23, J4.26, J4.9, R31.1, R32.1, R4.1, R5.2, R9.2, U2.2, U3.1, U3.10, U3.11, U3.20, U3.4, U3.PAD, U7.2
- net I_SENSE: no longer C12.1, R5.1, U3.8
- net LED_CTRL: no longer U2.4
- net MISO: no longer J2.7
- net MOSI: no longer J2.3
- net PB22: no longer J2.2
- net RX0: no longer J1.6
- net SCK: no longer J2.5
- net SCL_BUFF: no longer J4.12
- net SDA_BUFF: no longer J4.13
- net TX0: no longer J1.7
Routing:
- net BIAS_V: track 112.5 -> 0.00 mm, vias 5 -> 0
- net BIAS_GND: track 87.8 -> 0.00 mm, vias 2 -> 0
- net LED_V: track 82.5 -> 0.00 mm, vias 1 -> 0
- net LED_GND: track 77.7 -> 0.00 mm, vias 1 -> 0
- net MA1: track 41.5 -> 0.00 mm, vias 2 -> 0
- net 5V_S: track 124.8 -> 85.4 mm, vias 14 -> 10
- net C_3V3: track 32.7 -> 0.00 mm
- net +5V: track 90.0 -> 57.4 mm, vias 4 -> 3
- net MA2: track 32.4 -> 0.00 mm, vias 2 -> 0
- net C_SDA0: track 32.3 -> 0.00 mm
- net MB1: track 29.9 -> 0.00 mm
- net C_SCL0: track 29.9 -> 0.00 mm
- net CAM_CLK: track 29.6 -> 0.00 mm
- net CAM1_C_N: track 26.0 -> 0.00 mm
- net CAM1_C_P: track 25.9 -> 0.00 mm
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