File: CAD/Eagle/STARduino/starduino.sch (EAGLE design)
At the start: 97 parts, among them J1 J30J-9J30, J2 MICRO_SD, J3 J30J-15J30, J4 J30J-31J30, Q2 BSS8402DW, Q3 BSS8402DW, Q4 DMMT5401, Q5 DMG2305UX, U1 SSCMNNN015PA2A3, U10 MC14504BDTG, U11 MAX31725MTA+, U12 TCA9535_RTW_24, U13 BMX055, U15 MC74VHC1GT125, U16 PCA9515A, U17 PCA9306DCT, U2 LT3465/A, U3 LTC3112FE, U4 DS3231MZ+, U5 MT25QL01GBBB8ESF-0AAT, U6 ATSAMD21G18, U7 MIC5319, U8 ADXL375BCCZ

Commit message: STARduino and Datalogger
Parts:
- removed C11: 10pF, resistor:C-USC0603
- removed C12, C18: 47pF, resistor:C-USC0603
- removed C13, C29, C6: 100nF, resistor:C-USC0603
- removed C14: 680pF, resistor:C-USC0603
- removed C15, C28, C3, C4, C42: 1uF, resistor:C-USC0603
- removed C19: 47uF, resistor:C-USC1210
- removed C2: 22uF, resistor:C-USC1206
- removed C30: 2.2uF, resistor:C-USC0603
- removed D4: B0520LW-7-F, CM_diodes:SCHOTTKY-DIODESOD123
- removed J1: J30J-9J30, CM_J30J:J30J-9J30
- removed J2: MICRO_SD, NR_connectors:MICRO_SD
- removed L1: 22uH, AR_passives:INDUCTOR-VLF504012MT
- removed L2: 4.7uH, CM_passives:SRP5030T
- removed Q4: DMMT5401, transistor-pnp:DMMT5401
- removed Q5: DMG2305UX, transistor-fet:DMG2305UX
- removed R10, R31: 10k, resistor:R-US_R0603
- removed R32: 47k, resistor:R-US_R0603
- removed R33: 1M, resistor:R-US_R0603
- removed R4: 6.2, resistor:R-US_R0603
- removed R5, R6: 33k, resistor:R-US_R0603
- removed R8: 845k, resistor:R-US_R0603
- removed R9: 158k, resistor:R-US_R0603
- removed U2: LT3465/A, AR_IC:LT3465/A
- removed U3: LTC3112FE, CM_IC:LTC3112FE
- removed U7: MIC5319, CM_IC:MIC5319
Connections:
- removed net BIAS_GND: J4.3
- removed net BIAS_V: J4.4
- removed net CAM1_C_N: J4.24
- removed net CAM1_C_P: J4.25
- removed net CAM1_D0_N: J4.18
- removed net CAM1_D0_P: J4.19
- removed net CAM1_D1_N: J4.21
- removed net CAM1_D1_P: J4.22
- removed net CAM_CLK: J4.28
- removed net CAM_GPIO: J4.27
- removed net C_3V3: J4.31
- removed net C_SCL0: J4.29
- removed net C_SDA0: J4.30
- removed net FB_5: C11.2, C14.2, R10.1, R8.2, R9.1, U3.FB
- removed net LED_GND: J4.2, R4.2, U2.FB
- removed net LED_V: C15.1, J4.1, U2.V_OUT
- removed net MA1: J4.5
- removed net MA2: J4.6
- removed net MB1: J4.7
- removed net MB2: J4.8
- removed net N$1: Q4.C2, Q5.G, R32.2
- removed net N$11: C14.1, R6.1
- removed net N$12: C11.1, R6.2, U3.COMP
- removed net N$15: L1.2, U2.SW
- removed net N$2: Q4.B1, Q4.B2, Q4.C1, R31.2
- removed net N$3: R33.1, U3.PWM/SYNC
- removed net N$39: C6.1, L2.P$1, U3.SW1
- removed net N$40: C13.1, L2.P$2, U3.SW2
- removed net N$41: C6.2, U3.BST1
- removed net N$42: C13.2, U3.BST2
- removed net N$43: C4.1, D4.C, R33.2, U3.VCC
- removed net N$48: C18.2, R10.2
- removed net N$9: C29.1, U7.BYP
- removed net VCC: C2.1, C42.1, J1.1, J1.2, U3.RUN, U3.VIN
- net +3V3: no longer C30.1, J2.SD_VDD, U7.VOUT
- net +5V: no longer C18.1, C19.1, D4.A, Q4.E1, Q5.S, R8.1, U3.VOUT
- net 5V_S: no longer C28.1, C3.1, L1.1, Q4.E2, Q5.D, U2.VCC, U7.EN, U7.VIN
- net EXTERNAL_3V3: no longer J4.15
- net GND: no longer C12.2, C15.2, C19.2, C2.2, C28.2, C29.2, C3.2, C30.2, C4.2, C42.2, J1.3, J1.4, J1.5, J2.GND@1, J2.GND@2, J2.GND@3, J2.SD_GND, J4.14, J4.17, J4.20, J4.23, J4.26, J4.9, R31.1, R32.1, R4.1, R5.2, R9.2, U2.GND, U3.GND, U3.OVP, U7.GND
- net I_SENSE: no longer C12.1, R5.1, U3.IOUT
- net LED_CTRL: no longer U2.EN
- net MISO: no longer J2.DATA_OUT
- net MOSI: no longer J2.DATA_IN
- net PB22: no longer J2.CS
- net RX0: no longer J1.6
- net SCK: no longer J2.SCLK
- net SCL_BUFF: no longer J4.12
- net SDA_BUFF: no longer J4.13
- net TX0: no longer J1.7
Other:
- note added: "3.3V SUPPLY"
- note removed: "3.3V LDO"
- note removed: "5V PROTECT"
- note removed: "HERMES MDM"
- note removed: "MICRO SD CARD"
