File: CAD/Eagle/Datalogger/datalogger.sch (EAGLE design)
At the start: 8 parts, among them U1 MT25QL01GBBB8ESF-0AAT

Commit message: datalogger, mostly done
Parts:
- added U$4: SSL.3IN_SILK, images:SSL.3IN_SILK
Connections:
- net DATA+1 renamed DATA1_P
- net DATA+2 renamed DATA2_P
- net DATA-1 renamed DATA1_N
- removed net DATA+3: CONNECTOR.14, U$3.DATA+1
- removed net DATA+4: CONNECTOR.16, U$3.DATA+2
- removed net DATA-2: CONNECTOR.26, U$2.DATA-2
- removed net DATA-3: CONNECTOR.31, U$3.DATA-1
- removed net DATA-4: CONNECTOR.30, U$3.DATA-2
- new net DATA2_N: CONNECTOR.24, U$2.DATA-2
- new net DATA3_N: CONNECTOR.30, U$3.DATA-1
- new net DATA3_P: CONNECTOR.31, U$3.DATA+1
- new net DATA4_N: CONNECTOR.16, U$3.DATA-2
- new net DATA4_P: CONNECTOR.15, U$3.DATA+2
- new net N$10: CONNECTOR.11
- new net N$11: CONNECTOR.12
- new net N$12: CONNECTOR.13
- new net N$2: CONNECTOR.3
- new net N$3: CONNECTOR.4
- new net N$4: CONNECTOR.5
- new net N$5: CONNECTOR.6
- new net N$6: CONNECTOR.7
- new net N$7: CONNECTOR.8
- new net N$8: CONNECTOR.9
- new net N$9: CONNECTOR.10
- net GND: now also CONNECTOR.14, CONNECTOR.26; no longer CONNECTOR.15, CONNECTOR.24
Changed lines of the file:
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@@
 <class number="0" name="default" width="0" drill="0">
+</class>
+<class number="1" name="diff_pair" width="0.4064" drill="0">
 </class>
 </classes>
@@
 <part name="GND5" library="supply1" deviceset="GND" device=""/>
 <part name="+3V2" library="supply1" deviceset="+3V3" device=""/>
+<part name="U$4" library="images" deviceset="SSL" device=".3IN_SILK"/>
 </parts>
 <sheets>
@@
 <attribute name="VALUE" x="40.64" y="185.42" size="1.778" layer="96" rot="R270"/>
 </instance>
+<instance part="U$4" gate="G$1" x="-2.54" y="96.52"/>
 </instances>
 <busses>
@@
 <net name="GND" class="0">
 <segment>
-<pinref part="CONNECTOR" gate="G$1" pin="15"/>
-<wire x1="38.1" y1="58.42" x2="33.02" y2="58.42" width="0.1524" layer="91"/>
-<label x="33.02" y="58.42" size="1.778" layer="95" rot="R180" xref="yes"/>
-</segment>
-<segment>
-<pinref part="U$2" gate="G$1" pin="GND1"/>
 <pinref part="GND1" gate="1" pin="GND"/>
-<wire x1="30.48" y1="254" x2="15.24" y2="254" width="0.1524" layer="91"/>
 <wire x1="15.24" y1="254" x2="15.24" y2="241.3" width="0.1524" layer="91"/>
 <pinref part="U$2" gate="G$1" pin="GND2"/>
 <wire x1="15.24" y1="241.3" x2="15.24" y2="231.14" width="0.1524" layer="91"/>
 <wire x1="30.48" y1="241.3" x2="15.24" y2="241.3" width="0.1524" layer="91"/>
+<pinref part="U$2" gate="G$1" pin="GND1"/>
+<wire x1="30.48" y1="254" x2="15.24" y2="254" width="0.1524" layer="91"/>
 </segment>
 <segment>
@@
 </segment>
 <segment>
-<pinref part="CONNECTOR" gate="G$1" pin="24"/>
-<wire x1="48.26" y1="91.44" x2="53.34" y2="91.44" width="0.1524" layer="91"/>
-<label x="53.34" y="91.44" size="1.778" layer="95" xref="yes"/>
+<pinref part="CONNECTOR" gate="G$1" pin="26"/>
+<wire x1="48.26" y1="81.28" x2="53.34" y2="81.28" width="0.1524" layer="91"/>
+<label x="53.34" y="81.28" size="1.778" layer="95" xref="yes"/>
+</segment>
+<segment>
+<pinref part="CONNECTOR" gate="G$1" pin="14"/>
+<wire x1="38.1" y1="63.5" x2="33.02" y2="63.5" width="0.1524" layer="91"/>
+<label x="33.02" y="63.5" size="1.778" layer="95" rot="R180" xref="yes"/>
 </segment>
 </net>
@@
 </segment>
 </net>
-<net name="DATA+1" class="0">
+<net name="DATA1_P" class="0">
 <segment>
 <pinref part="U$2" gate="G$1" pin="DATA+1"/>
@@
 </segment>
 </net>
-<net name="DATA-1" class="0">
+<net name="DATA1_N" class="0">
 <segment>
 <pinref part="U$2" gate="G$1" pin="DATA-1"/>
@@
 </segment>
 </net>
-<net name="DATA+2" class="0">
+<net name="DATA2_P" class="0">
 <segment>
 <pinref part="U$2" gate="G$1" pin="DATA+2"/>
@@
 </segment>
 </net>
-<net name="DATA-2" class="0">
+<net name="DATA2_N" class="0">
 <segment>
 <pinref part="U$2" gate="G$1" pin="DATA-2"/>
@@
 </segment>
 <segment>
-<pinref part="CONNECTOR" gate="G$1" pin="26"/>
-<wire x1="48.26" y1="81.28" x2="53.34" y2="81.28" width="0.1524" layer="91"/>
-<label x="53.34" y="81.28" size="1.778" layer="95" xref="yes"/>
-</segment>
-</net>
-<net name="DATA+3" class="0">
+<pinref part="CONNECTOR" gate="G$1" pin="24"/>
+<wire x1="48.26" y1="91.44" x2="53.34" y2="91.44" width="0.1524" layer="91"/>
+<label x="53.34" y="91.44" size="1.778" layer="95" xref="yes"/>
+</segment>
+</net>
+<net name="DATA3_P" class="0">
 <segment>
 <pinref part="U$3" gate="G$1" pin="DATA+1"/>
@@
 </segment>
 <segment>
-<pinref part="CONNECTOR" gate="G$1" pin="14"/>
-<wire x1="38.1" y1="63.5" x2="33.02" y2="63.5" width="0.1524" layer="91"/>
-<label x="33.02" y="63.5" size="1.778" layer="95" rot="R180" xref="yes"/>
-</segment>
-</net>
-<net name="DATA-3" class="0">
+<pinref part="CONNECTOR" gate="G$1" pin="31"/>
+<wire x1="48.26" y1="55.88" x2="53.34" y2="55.88" width="0.1524" layer="91"/>
+<label x="53.34" y="55.88" size="1.778" layer="95" xref="yes"/>
+</segment>
+</net>
+<net name="DATA3_N" class="0">
 <segment>
 <pinref part="U$3" gate="G$1" pin="DATA-1"/>
@@
 </segment>
 <segment>
-<pinref part="CONNECTOR" gate="G$1" pin="31"/>
-<wire x1="48.26" y1="55.88" x2="53.34" y2="55.88" width="0.1524" layer="91"/>
-<label x="53.34" y="55.88" size="1.778" layer="95" xref="yes"/>
-</segment>
-</net>
-<net name="DATA+4" class="0">
+<pinref part="CONNECTOR" gate="G$1" pin="30"/>
+<wire x1="48.26" y1="60.96" x2="53.34" y2="60.96" width="0.1524" layer="91"/>
+<label x="53.34" y="60.96" size="1.778" layer="95" xref="yes"/>
+</segment>
+</net>
+<net name="DATA4_P" class="0">
+<segment>
+<pinref part="U$3" gate="G$1" pin="DATA+2"/>
+<wire x1="99.06" y1="236.22" x2="93.98" y2="236.22" width="0.1524" layer="91"/>
+<label x="93.98" y="236.22" size="1.016" layer="95" rot="R180" xref="yes"/>
+</segment>
+<segment>
+<pinref part="CONNECTOR" gate="G$1" pin="15"/>
+<wire x1="38.1" y1="58.42" x2="33.02" y2="58.42" width="0.1524" layer="91"/>
+<label x="33.02" y="58.42" size="1.778" layer="95" rot="R180" xref="yes"/>
+</segment>
+</net>
+<net name="DATA4_N" class="0">
+<segment>
+<pinref part="U$3" gate="G$1" pin="DATA-2"/>
+<wire x1="129.54" y1="241.3" x2="134.62" y2="241.3" width="0.1524" layer="91"/>
+<label x="134.62" y="241.3" size="1.016" layer="95" xref="yes"/>
+</segment>
 <segment>
 <pinref part="CONNECTOR" gate="G$1" pin="16"/>
 <wire x1="38.1" y1="53.34" x2="33.02" y2="53.34" width="0.1524" layer="91"/>
 <label x="33.02" y="53.34" size="1.778" layer="95" rot="R180" xref="yes"/>
-</segment>
-<segment>
-<pinref part="U$3" gate="G$1" pin="DATA+2"/>
-<wire x1="99.06" y1="236.22" x2="93.98" y2="236.22" width="0.1524" layer="91"/>
-<label x="93.98" y="236.22" size="1.016" layer="95" rot="R180" xref="yes"/>
-</segment>
-</net>
-<net name="DATA-4" class="0">
-<segment>
-<pinref part="U$3" gate="G$1" pin="DATA-2"/>
-<wire x1="129.54" y1="241.3" x2="134.62" y2="241.3" width="0.1524" layer="91"/>
-<label x="134.62" y="241.3" size="1.016" layer="95" xref="yes"/>
-</segment>
-<segment>
-<pinref part="CONNECTOR" gate="G$1" pin="30"/>
-<wire x1="48.26" y1="60.96" x2="53.34" y2="60.96" width="0.1524" layer="91"/>
-<label x="53.34" y="60.96" size="1.778" layer="95" xref="yes"/>
 </segment>
 </net>
@@
 </segment>
 </net>
+<net name="N$2" class="0">
+<segment>
+<pinref part="CONNECTOR" gate="G$1" pin="3"/>
+<wire x1="38.1" y1="119.38" x2="33.02" y2="119.38" width="0.1524" layer="91"/>
+</segment>
+</net>
+<net name="N$3" class="0">
+<segment>
+<pinref part="CONNECTOR" gate="G$1" pin="4"/>
+<wire x1="38.1" y1="114.3" x2="33.02" y2="114.3" width="0.1524" layer="91"/>
+</segment>
+</net>
+<net name="N$4" class="0">
+<segment>
+<pinref part="CONNECTOR" gate="G$1" pin="5"/>
+<wire x1="38.1" y1="109.22" x2="33.02" y2="109.22" width="0.1524" layer="91"/>
+</segment>
+</net>
+<net name="N$5" class="0">
+<segment>
+<pinref part="CONNECTOR" gate="G$1" pin="6"/>
+<wire x1="38.1" y1="104.14" x2="33.02" y2="104.14" width="0.1524" layer="91"/>
+</segment>
+</net>
+<net name="N$6" class="0">
+<segment>
+<pinref part="CONNECTOR" gate="G$1" pin="7"/>
+<wire x1="38.1" y1="99.06" x2="33.02" y2="99.06" width="0.1524" layer="91"/>
+</segment>
+</net>
+<net name="N$7" class="0">
+<segment>
+<pinref part="CONNECTOR" gate="G$1" pin="8"/>
+<wire x1="38.1" y1="93.98" x2="33.02" y2="93.98" width="0.1524" layer="91"/>
+</segment>
+</net>
+<net name="N$8" class="0">
+<segment>
+<pinref part="CONNECTOR" gate="G$1" pin="9"/>
+<wire x1="38.1" y1="88.9" x2="33.02" y2="88.9" width="0.1524" layer="91"/>
+</segment>
+</net>
+<net name="N$9" class="0">
+<segment>
+<pinref part="CONNECTOR" gate="G$1" pin="10"/>
+<wire x1="38.1" y1="83.82" x2="33.02" y2="83.82" width="0.1524" layer="91"/>
+</segment>
+</net>
+<net name="N$10" class="0">
+<segment>
+<pinref part="CONNECTOR" gate="G$1" pin="11"/>
+<wire x1="38.1" y1="78.74" x2="33.02" y2="78.74" width="0.1524" layer="91"/>
+</segment>
+</net>
+<net name="N$11" class="0">
+<segment>
+<pinref part="CONNECTOR" gate="G$1" pin="12"/>
+<wire x1="38.1" y1="73.66" x2="33.02" y2="73.66" width="0.1524" layer="91"/>
+</segment>
+</net>
+<net name="N$12" class="0">
+<segment>
+<pinref part="CONNECTOR" gate="G$1" pin="13"/>
+<wire x1="38.1" y1="68.58" x2="33.02" y2="68.58" width="0.1524" layer="91"/>
+</segment>
+</net>

Commit message: Datalogger v1 final
Connections:
- removed net N$11: CONNECTOR.12
- net DATA2_N: now also CONNECTOR.25; no longer CONNECTOR.24
- net DATA2_P: now also CONNECTOR.24; no longer CONNECTOR.25
- net GND: now also CONNECTOR.12
Changed lines of the file:
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@@
 <label x="33.02" y="63.5" size="1.778" layer="95" rot="R180" xref="yes"/>
+</segment>
+<segment>
+<pinref part="CONNECTOR" gate="G$1" pin="12"/>
+<wire x1="38.1" y1="73.66" x2="33.02" y2="73.66" width="0.1524" layer="91"/>
+<label x="33.02" y="73.66" size="1.778" layer="95" rot="R180" xref="yes"/>
 </segment>
 </net>
@@
 </segment>
 <segment>
+<pinref part="CONNECTOR" gate="G$1" pin="24"/>
+<wire x1="48.26" y1="91.44" x2="53.34" y2="91.44" width="0.1524" layer="91"/>
+<label x="53.34" y="91.44" size="1.778" layer="95" xref="yes"/>
+</segment>
+</net>
+<net name="DATA2_N" class="0">
+<segment>
+<pinref part="U$2" gate="G$1" pin="DATA-2"/>
+<wire x1="60.96" y1="241.3" x2="66.04" y2="241.3" width="0.1524" layer="91"/>
+<label x="66.04" y="241.3" size="1.016" layer="95" xref="yes"/>
+</segment>
+<segment>
 <pinref part="CONNECTOR" gate="G$1" pin="25"/>
 <wire x1="48.26" y1="86.36" x2="53.34" y2="86.36" width="0.1524" layer="91"/>
 <label x="53.34" y="86.36" size="1.778" layer="95" xref="yes"/>
-</segment>
-</net>
-<net name="DATA2_N" class="0">
-<segment>
-<pinref part="U$2" gate="G$1" pin="DATA-2"/>
-<wire x1="60.96" y1="241.3" x2="66.04" y2="241.3" width="0.1524" layer="91"/>
-<label x="66.04" y="241.3" size="1.016" layer="95" xref="yes"/>
-</segment>
-<segment>
-<pinref part="CONNECTOR" gate="G$1" pin="24"/>
-<wire x1="48.26" y1="91.44" x2="53.34" y2="91.44" width="0.1524" layer="91"/>
-<label x="53.34" y="91.44" size="1.778" layer="95" xref="yes"/>
 </segment>
 </net>
@@
 </segment>
 </net>
-<net name="N$11" class="0">
-<segment>
-<pinref part="CONNECTOR" gate="G$1" pin="12"/>
-<wire x1="38.1" y1="73.66" x2="33.02" y2="73.66" width="0.1524" layer="91"/>
-</segment>
-</net>
