File: STAR/Eagle/STARduino/starduino.sch (EAGLE design)
At the start: 63 parts, among them J3 J30J-15J30, J4 J30J-31J30, Q2 BSS8402DW, Q3 BSS8402DW, U1 SSCMNNN015PA2A3, U10 MC14504BDTG, U11 MAX31725MTA+, U12 TCA9535_RTW_24, U13 BMX055, U15 MC74VHC1GT125, U16 PCA9515A, U17 PCA9306DCT, U4 DS3231MZ+, U5 MT25QL01GBBB8ESF-0AAT, U6 ATSAMD21G18, U8 ADXL375BCCZ

Commit message: Added STARduino voltage regulation
Parts:
- removed L3, L6: 10uH, AR_passives:INDUCTOR-0603
- added C11, C6: 4.7uF, resistor:C-USC0603
- added C12: 1uF, resistor:C-USC0603
- added C13, C14: 1nF, resistor:C-USC0603
- added C15, C16: 100nF, resistor:C-USC0603
- added C17, C19: 4.7pF, rcl:C-USC0603
- added C18, C23: 47uF, resistor:C-USC1210
- added FB2: BLM18KG221BH1D, AR_passives:FERRITE_BEAD-0603
- added L1: 8.5uH, AR_passives:INDUCTOR744314850
- added L2: 7.8uH, AR_passives:INDUCTORSRP-1250
- added R2: 24.3k, resistor:R-US_R0603
- added R4, R5: 1M, resistor:R-US_R0603
- added R6: 560k, resistor:R-US_R0603
- added R7: 176k, resistor:R-US_R0603
- added R8: 820k, resistor:R-US_R0603
- added R9: 154k, resistor:R-US_R0603
- added U18: LT8616, AR_IC:LT8616
- C21: value 10uF -> 100nF
- C22: value 100nF -> 10uF
Connections:
- new net N$1: R2.1, U18.RT
- new net N$11: C16.1, U18.BOOST2
- new net N$12: C15.1, U18.BOOST1
- new net N$13: C15.2
- new net N$14: L1.1, U18.SW1
- new net N$16: C16.2
- new net N$17: L2.1, U18.SW2
- new net N$20: R4.1, U18.PG1
- new net N$21: R5.1, U18.PG2
- new net N$22: C17.2, R6.2, R7.1, U18.FB1
- new net N$3: C12.1, U18.INTVCC
- new net N$37: C19.2, R8.2, R9.1, U18.FB2
- new net N$9: C14.1, U18.SS2
- new net VDD: C11.1, C6.1, U18.EN1, U18.EN2, U18.VIN1, U18.VIN2
- net +3V3: now also C1.1, C17.1, C18.1, C2.1, C20.1, FB2.P$2, L1.2, R4.2, R6.1, U18.BIAS, U6.VCC, U6.VDDIO1, U6.VDDIO2; no longer L3.1, L6.2
- net +5V: now also C19.1, C23.1, L2.2, R5.2, R8.1
- net GND: now also C11.2, C12.2, C13.2, C14.2, C18.2, C23.2, C6.2, R2.2, R7.2, R9.2, U18.GND, U18.SYNC
- net N$4: now also C13.1, U18.SS1; no longer C1.1, C2.1, C20.1, L3.2, U6.VCC, U6.VDDIO1, U6.VDDIO2
- net VREFA: now also FB2.P$1; no longer L6.1
Other:
- note added: "VOLTAGE REGULATION"
- note removed: "3.3V SUPPLY"
- note removed: "5V SUPPLY"
- moved on the sheet: C20, J3, J4, Q2N, Q2P, R13, R15
