File: STAR/Eagle/STARduino/starduino.sch (EAGLE design)
At the start: 76 parts, among them J1 J30J-25, Q2 BSS8402DW, U1 SSCMNNN015PA2A3, U10 MC14504BDTG, U11 MAX31725MTA+, U12 TCA9535_RTW_24, U13 BMX055, U15 MC74VHC1GT125, U16 PCA9515A, U17 PCA9306DCT, U18 LT8616, U4 DS3231MZ+, U6 ATSAMD21G18, U8 ADXL375BCCZ

Commit message: STARduino
Connections:
- net +3V3: now also J1.1, J1.3; no longer J1.14
- net +5V: now also J1.20, J1.5, J1.6, J1.8; no longer J1.15, J1.16, J1.17, J1.18
- net GND: now also J1.7; no longer J1.20, J1.25
- net MISO: now also J1.15, J1.17; no longer J1.3, J1.4
- net MOSI: now also J1.14, J1.4; no longer J1.5, J1.6
- net SCK: now also J1.16, J1.18; no longer J1.7, J1.8
- net VDD: now also J1.25; no longer J1.1
Changed lines of the file:
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@@
 <part name="VDD1" library="supply1" deviceset="VDD" device=""/>
 <part name="J1" library="CM_J30J" deviceset="J30J-25" device=""/>
-<part name="GND42" library="supply1" deviceset="GND" device=""/>
 </parts>
 <sheets>
@@
 <instance part="VDD1" gate="G$1" x="12.7" y="144.78"/>
 <instance part="J1" gate="G$1" x="220.98" y="111.76"/>
-<instance part="GND42" gate="1" x="231.14" y="76.2"/>
 </instances>
 <busses>
@@
 </segment>
 <segment>
-<pinref part="J1" gate="G$1" pin="14"/>
-<wire x1="226.06" y1="139.7" x2="228.6" y2="139.7" width="0.1524" layer="91"/>
-<label x="228.6" y="139.7" size="1.016" layer="95" xref="yes"/>
+<pinref part="J1" gate="G$1" pin="1"/>
+<wire x1="215.9" y1="142.24" x2="213.36" y2="142.24" width="0.1524" layer="91"/>
+<label x="213.36" y="142.24" size="1.016" layer="95" rot="R180" xref="yes"/>
+</segment>
+<segment>
+<pinref part="J1" gate="G$1" pin="3"/>
+<wire x1="215.9" y1="132.08" x2="213.36" y2="132.08" width="0.1524" layer="91"/>
+<label x="213.36" y="132.08" size="1.016" layer="95" rot="R180" xref="yes"/>
 </segment>
 </net>
@@
 <segment>
 <pinref part="J1" gate="G$1" pin="22"/>
-<wire x1="226.06" y1="99.06" x2="231.14" y2="99.06" width="0.1524" layer="91"/>
-<wire x1="231.14" y1="99.06" x2="231.14" y2="93.98" width="0.1524" layer="91"/>
+<wire x1="226.06" y1="99.06" x2="228.6" y2="99.06" width="0.1524" layer="91"/>
+<label x="228.6" y="99.06" size="1.016" layer="95" xref="yes"/>
+</segment>
+<segment>
 <pinref part="J1" gate="G$1" pin="23"/>
-<wire x1="231.14" y1="93.98" x2="231.14" y2="88.9" width="0.1524" layer="91"/>
-<wire x1="231.14" y1="88.9" x2="231.14" y2="83.82" width="0.1524" layer="91"/>
-<wire x1="231.14" y1="83.82" x2="231.14" y2="78.74" width="0.1524" layer="91"/>
-<wire x1="226.06" y1="93.98" x2="231.14" y2="93.98" width="0.1524" layer="91"/>
+<wire x1="226.06" y1="93.98" x2="228.6" y2="93.98" width="0.1524" layer="91"/>
+<label x="228.6" y="93.98" size="1.016" layer="95" xref="yes"/>
+</segment>
+<segment>
 <pinref part="J1" gate="G$1" pin="24"/>
-<wire x1="226.06" y1="88.9" x2="231.14" y2="88.9" width="0.1524" layer="91"/>
-<pinref part="J1" gate="G$1" pin="25"/>
-<wire x1="226.06" y1="83.82" x2="231.14" y2="83.82" width="0.1524" layer="91"/>
-<pinref part="GND42" gate="1" pin="GND"/>
-<pinref part="J1" gate="G$1" pin="20"/>
-<wire x1="226.06" y1="109.22" x2="231.14" y2="109.22" width="0.1524" layer="91"/>
-<wire x1="231.14" y1="109.22" x2="231.14" y2="106.68" width="0.1524" layer="91"/>
+<wire x1="226.06" y1="88.9" x2="228.6" y2="88.9" width="0.1524" layer="91"/>
+<label x="228.6" y="88.9" size="1.016" layer="95" xref="yes"/>
+</segment>
+<segment>
+<pinref part="J1" gate="G$1" pin="7"/>
+<wire x1="215.9" y1="111.76" x2="213.36" y2="111.76" width="0.1524" layer="91"/>
+<label x="213.36" y="111.76" size="1.016" layer="95" rot="R180" xref="yes"/>
+</segment>
+<segment>
 <pinref part="J1" gate="G$1" pin="21"/>
-<wire x1="231.14" y1="104.14" x2="231.14" y2="99.06" width="0.1524" layer="91"/>
-<wire x1="226.06" y1="104.14" x2="231.14" y2="104.14" width="0.1524" layer="91"/>
-<wire x1="231.14" y1="104.14" x2="231.14" y2="106.68" width="0.1524" layer="91"/>
+<wire x1="226.06" y1="104.14" x2="228.6" y2="104.14" width="0.1524" layer="91"/>
+<label x="228.6" y="104.14" size="1.016" layer="95" xref="yes"/>
 </segment>
 </net>
@@
 </segment>
 <segment>
-<pinref part="J1" gate="G$1" pin="3"/>
-<wire x1="215.9" y1="132.08" x2="213.36" y2="132.08" width="0.1524" layer="91"/>
-<pinref part="J1" gate="G$1" pin="4"/>
-<wire x1="215.9" y1="127" x2="213.36" y2="127" width="0.1524" layer="91"/>
-<wire x1="213.36" y1="132.08" x2="213.36" y2="127" width="0.1524" layer="91"/>
-<label x="213.36" y="132.08" size="1.016" layer="95" rot="R180" xref="yes"/>
+<pinref part="J1" gate="G$1" pin="15"/>
+<wire x1="226.06" y1="134.62" x2="228.6" y2="134.62" width="0.1524" layer="91"/>
+<label x="228.6" y="134.62" size="1.016" layer="95" xref="yes"/>
+</segment>
+<segment>
+<pinref part="J1" gate="G$1" pin="17"/>
+<wire x1="226.06" y1="124.46" x2="228.6" y2="124.46" width="0.1524" layer="91"/>
+<label x="228.6" y="124.46" size="1.016" layer="95" xref="yes"/>
 </segment>
 </net>
@@
 </segment>
 <segment>
-<pinref part="J1" gate="G$1" pin="5"/>
-<wire x1="215.9" y1="121.92" x2="213.36" y2="121.92" width="0.1524" layer="91"/>
-<pinref part="J1" gate="G$1" pin="6"/>
-<wire x1="215.9" y1="116.84" x2="213.36" y2="116.84" width="0.1524" layer="91"/>
-<wire x1="213.36" y1="121.92" x2="213.36" y2="116.84" width="0.1524" layer="91"/>
-<label x="213.36" y="121.92" size="1.016" layer="95" rot="R180" xref="yes"/>
+<pinref part="J1" gate="G$1" pin="14"/>
+<wire x1="226.06" y1="139.7" x2="228.6" y2="139.7" width="0.1524" layer="91"/>
+<label x="228.6" y="139.7" size="1.016" layer="95" xref="yes"/>
+</segment>
+<segment>
+<pinref part="J1" gate="G$1" pin="4"/>
+<wire x1="215.9" y1="127" x2="213.36" y2="127" width="0.1524" layer="91"/>
+<label x="213.36" y="127" size="1.016" layer="95" rot="R180" xref="yes"/>
 </segment>
 </net>
@@
 </segment>
 <segment>
-<pinref part="J1" gate="G$1" pin="7"/>
-<wire x1="215.9" y1="111.76" x2="213.36" y2="111.76" width="0.1524" layer="91"/>
-<pinref part="J1" gate="G$1" pin="8"/>
-<wire x1="215.9" y1="106.68" x2="213.36" y2="106.68" width="0.1524" layer="91"/>
-<wire x1="213.36" y1="111.76" x2="213.36" y2="106.68" width="0.1524" layer="91"/>
-<label x="213.36" y="111.76" size="1.016" layer="95" rot="R180" xref="yes"/>
+<pinref part="J1" gate="G$1" pin="16"/>
+<wire x1="228.6" y1="129.54" x2="226.06" y2="129.54" width="0.1524" layer="91"/>
+<label x="228.6" y="129.54" size="1.016" layer="95" xref="yes"/>
+</segment>
+<segment>
+<pinref part="J1" gate="G$1" pin="18"/>
+<wire x1="226.06" y1="119.38" x2="228.6" y2="119.38" width="0.1524" layer="91"/>
+<label x="228.6" y="119.38" size="1.016" layer="95" xref="yes"/>
 </segment>
 </net>
@@
 </segment>
 <segment>
-<pinref part="J1" gate="G$1" pin="17"/>
-<wire x1="226.06" y1="124.46" x2="228.6" y2="124.46" width="0.1524" layer="91"/>
-<wire x1="228.6" y1="124.46" x2="228.6" y2="119.38" width="0.1524" layer="91"/>
-<pinref part="J1" gate="G$1" pin="18"/>
-<wire x1="226.06" y1="119.38" x2="228.6" y2="119.38" width="0.1524" layer="91"/>
-<pinref part="J1" gate="G$1" pin="15"/>
-<wire x1="226.06" y1="134.62" x2="228.6" y2="134.62" width="0.1524" layer="91"/>
-<wire x1="228.6" y1="134.62" x2="228.6" y2="129.54" width="0.1524" layer="91"/>
-<pinref part="J1" gate="G$1" pin="16"/>
-<wire x1="228.6" y1="129.54" x2="228.6" y2="124.46" width="0.1524" layer="91"/>
-<wire x1="228.6" y1="129.54" x2="226.06" y2="129.54" width="0.1524" layer="91"/>
 <pinref part="J1" gate="G$1" pin="19"/>
 <wire x1="226.06" y1="114.3" x2="228.6" y2="114.3" width="0.1524" layer="91"/>
-<wire x1="228.6" y1="114.3" x2="228.6" y2="119.38" width="0.1524" layer="91"/>
-<label x="228.6" y="124.46" size="1.016" layer="95" xref="yes"/>
+<label x="228.6" y="114.3" size="1.016" layer="95" xref="yes"/>
+</segment>
+<segment>
+<pinref part="J1" gate="G$1" pin="20"/>
+<wire x1="226.06" y1="109.22" x2="228.6" y2="109.22" width="0.1524" layer="91"/>
+<label x="228.6" y="109.22" size="1.016" layer="95" xref="yes"/>
+</segment>
+<segment>
+<pinref part="J1" gate="G$1" pin="8"/>
+<wire x1="215.9" y1="106.68" x2="213.36" y2="106.68" width="0.1524" layer="91"/>
+<label x="213.36" y="106.68" size="1.016" layer="95" rot="R180" xref="yes"/>
+</segment>
+<segment>
+<pinref part="J1" gate="G$1" pin="6"/>
+<wire x1="215.9" y1="116.84" x2="213.36" y2="116.84" width="0.1524" layer="91"/>
+<label x="213.36" y="116.84" size="1.016" layer="95" rot="R180" xref="yes"/>
+</segment>
+<segment>
+<pinref part="J1" gate="G$1" pin="5"/>
+<wire x1="215.9" y1="121.92" x2="213.36" y2="121.92" width="0.1524" layer="91"/>
+<label x="213.36" y="121.92" size="1.016" layer="95" rot="R180" xref="yes"/>
 </segment>
 </net>
@@
 </segment>
 <segment>
-<pinref part="J1" gate="G$1" pin="1"/>
-<wire x1="215.9" y1="142.24" x2="213.36" y2="142.24" width="0.1524" layer="91"/>
-<label x="213.36" y="142.24" size="1.016" layer="95" rot="R180" xref="yes"/>
-</segment>
-</net>
+<pinref part="J1" gate="G$1" pin="25"/>
+<wire x1="226.06" y1="83.82" x2="228.6" y2="83.82" width="0.1524" layer="91"/>
+<label x="228.6" y="83.82" size="1.016" layer="95" xref="yes"/>
+</segment>
+</net>

Commit message: screws
Connections:
- removed net D: J1.10
- removed net N$27: J1.11
- removed net N$32: J1.12
- removed net N$36: J1.13
Other:
- note added: "CONNECTOR"
Changed lines of the file:
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@@
 <text x="482.6" y="419.1" size="5.08" layer="97">I2C BUFFER</text>
 <text x="434.34" y="317.5" size="5.08" layer="97">EXTERNAL POWER KILL</text>
-<wire x1="190.5" y1="170.18" x2="289.56" y2="170.18" width="0.3048" layer="97" style="shortdash"/>
+<wire x1="190.5" y1="170.18" x2="243.84" y2="170.18" width="0.3048" layer="97" style="shortdash"/>
+<wire x1="243.84" y1="170.18" x2="289.56" y2="170.18" width="0.3048" layer="97" style="shortdash"/>
 <wire x1="119.38" y1="170.18" x2="190.246" y2="170.18" width="0.3048" layer="97" style="shortdash"/>
 <wire x1="190.246" y1="170.18" x2="190.5" y2="170.18" width="0.3048" layer="97" style="shortdash"/>
@@
 <wire x1="190.246" y1="170.18" x2="190.246" y2="60.706" width="0.3048" layer="97" style="shortdash"/>
 <wire x1="190.246" y1="60.706" x2="5.08" y2="60.706" width="0.3048" layer="97" style="shortdash"/>
+<text x="197.358" y="157.226" size="5.08" layer="97">CONNECTOR</text>
+<wire x1="243.84" y1="170.18" x2="243.84" y2="60.96" width="0.3048" layer="97" style="shortdash"/>
+<wire x1="190.5" y1="60.96" x2="243.586" y2="60.96" width="0.3048" layer="97" style="shortdash"/>
 </plain>
 <instances>
@@
 </segment>
 </net>
-<net name="D" class="0">
-<segment>
-<pinref part="J1" gate="G$1" pin="10"/>
-<wire x1="215.9" y1="96.52" x2="213.36" y2="96.52" width="0.1524" layer="91"/>
-<label x="213.36" y="96.52" size="1.016" layer="95" rot="R180" xref="yes"/>
-</segment>
-</net>
 <net name="SD_STAR" class="0">
 <segment>
@@
 </segment>
 </net>
-<net name="N$27" class="0">
-<segment>
-<pinref part="J1" gate="G$1" pin="11"/>
-<wire x1="215.9" y1="91.44" x2="213.36" y2="91.44" width="0.1524" layer="91"/>
-<label x="213.36" y="91.44" size="1.016" layer="95" rot="R180" xref="yes"/>
-</segment>
-</net>
-<net name="N$32" class="0">
-<segment>
-<pinref part="J1" gate="G$1" pin="12"/>
-<wire x1="215.9" y1="86.36" x2="213.36" y2="86.36" width="0.1524" layer="91"/>
-<label x="213.36" y="86.36" size="1.016" layer="95" rot="R180" xref="yes"/>
-</segment>
-</net>
-<net name="N$36" class="0">
-<segment>
-<pinref part="J1" gate="G$1" pin="13"/>
-<wire x1="215.9" y1="81.28" x2="213.36" y2="81.28" width="0.1524" layer="91"/>
-<label x="213.36" y="81.28" size="1.016" layer="95" rot="R180" xref="yes"/>
-</segment>
-</net>

Commit message: external kill
Parts:
- removed Q2: BSS8402DW, transistor-fet:BSS8402DW
- removed R13: 100k, resistor:R-US_R0603
- removed R15: 191k, resistor:R-US_R0603
Connections:
- removed net DEBUG_5V: Q2P.D
- removed net EXTERNAL_KILL: Q2N.G, R13.1, U16.EN, U6.PA13/I2C/EIC/SCOM2PAD1+/TC2
- removed net N$38: Q2N.D, Q2P.G, R15.2
- net +5V: no longer Q2P.S, R15.1
- net GND: no longer Q2N.S, R13.2
Other:
- note removed: "DEBUG CUTOFF"
- moved on the sheet: J1

Commit message: misc board stuff
Parts:
- removed C33, C34, C35, C36, C37: 100nF, resistor:C-USC0603
- removed C41: 100pF, rcl:C-USC0603
- removed JP3: (no value), pinhead:PINHD-2X5
- removed R23: 4.7k, resistor:R-US_R0603
- removed R25, R27: 4.7k, rcl:R-US_R0603
- removed R26: 220k, rcl:R-US_R0603
- removed R28: 4.7k, SparkFun-Passives:RESISTOR-ARRAY0603-ARV
- removed R30: 10k, resistor:R-US_R0603
- removed U$1: STAR, images:STAR
- removed U$2: SSL.3IN_SILK, images:SSL.3IN_SILK
- removed U$3: CC2, NR_IC:CC2
- removed U15: MC74VHC1GT125, CM_IC:MC74VHC1GT125
- removed U16: PCA9515A, CM_IC:PCA9515A
- removed U17: PCA9306DCT, MotorDriver:PCA9306DCT
- removed U18: LT8616, AR_IC:LT8616
- added C24: 4.7pF, rcl:C-USC0603
- added C25: 47uF, resistor:C-USC1210
- added C26: 4.7uF, resistor:C-USC0603
- added C28, C30: 1nF, resistor:C-USC0603
- added C29: 100nF, resistor:C-USC0603
- added IMAG1: SSL.3IN_SILK, images:SSL.3IN_SILK
- added IMAG2: STAR, images:STAR
- added JP2: (no value), CM_passives:JUMPER-2PTH
- added R10: 4.7k, rcl:R-US_R0603
- added R11: 560k, resistor:R-US_R0603
- added R12, R14: 1M, resistor:R-US_R0603
- added R13: 176k, resistor:R-US_R0603
- added R15: 820k, resistor:R-US_R0603
- added U2: ATSAMD21G18, AR_mcu:ATSAMD21G18
- added U3: MAX31725MTA+, NR_IC:MAX31725MTA+
- added U5: DS3231MZ+, NR_IC:DS3231MZ+
- added U7: BMX055, NR_IC:BMX055
- added U9: TCA9535_RTW_24, MotorDriver:TCA9535_RTW_24
- C10: value 100nF -> 6.8pF
- C11: value 4.7uF -> 6.8pF
- C12: value 1uF -> 100nF
- C13, C14: value 1nF -> 100nF
- C15: value 100nF -> 10uF
- C17: value 4.7pF -> 1nF; device rcl:C-USC0603 -> resistor:C-USC0603
- C18: value 47uF -> 100nF; device resistor:C-USC1210 -> resistor:C-USC0603
- C19: value 4.7pF -> 100pF
- C21: value 100nF -> 220nF
- C22: value 10uF -> 100nF
- C23: value 47uF -> 4.7uF; device resistor:C-USC1210 -> resistor:C-USC0603
- C3: value 220nF -> 100nF
- C31: value 10uF -> 4.7pF; device resistor:C-USC0603 -> rcl:C-USC0603
- C32: value 100nF -> 47uF; device resistor:C-USC0603 -> resistor:C-USC1210
- C5: value 1nF -> 1uF
- C6: value 4.7uF -> 10uF
- C7, C8: value 6.8pF -> 100nF
- JP1: device CM_passives:JUMPER-2PTH -> pinhead:PINHD-2X5
- R1: value 330 -> 10k
- R16: value 3.6k -> 154k
- R17: value 6.8k -> 24.3k
- R2: value 24.3k -> 10k
- R3: value 10k -> 4.7k
- R4: value 1M -> 330
- R5: value 1M -> 3.6k
- R6: value 560k -> 6.8k
- R7: value 176k -> 4.7k; device resistor:R-US_R0603 -> SparkFun-Passives:RESISTOR-ARRAY0603-ARV
- R8: value 820k -> 220k; device resistor:R-US_R0603 -> rcl:R-US_R0603
- R9: value 154k -> 4.7k; device resistor:R-US_R0603 -> rcl:R-US_R0603
- U1: value SSCMNNN015PA2A3 -> PCA9515A; device NR_IC:SSCMNNN015PA2A3 -> CM_IC:PCA9515A
- U10: value MC14504BDTG -> PCA9306DCT; device MotorDriver:MC14504BDTG -> MotorDriver:PCA9306DCT
- U11: value MAX31725MTA+ -> CC2; device NR_IC:MAX31725MTA+ -> NR_IC:CC2
- U12: value TCA9535_RTW_24 -> SSCMNNN015PA2A3; device MotorDriver:TCA9535_RTW_24 -> NR_IC:SSCMNNN015PA2A3
- U13: value BMX055 -> LT8616; device NR_IC:BMX055 -> AR_IC:LT8616
- U4: value DS3231MZ+ -> MC74VHC1GT125; device NR_IC:DS3231MZ+ -> CM_IC:MC74VHC1GT125
- U6: value ATSAMD21G18 -> MC14504BDTG; device AR_mcu:ATSAMD21G18 -> MotorDriver:MC14504BDTG
Connections:
- net +3V3: now also C12.1, C13.1, C14.1, C15.1, C16.1, C21.2, C24.1, C25.1, C3.1, C4.1, FB1.P$2, FB2.P$1, JP1.1, R1.2, R11.1, R12.2, R2.2, R7A.2, R7B.2, R7C.2, R7D.2, U1.VCC, U10.VREF1, U12.VSUPPLY, U13.BIAS, U2.VCC, U2.VDDIO1, U2.VDDIO2, U3.VDD, U4.VIN, U5.VCC, U7.PS, U7.SDO2, U7.VDD, U7.VDDIO; no longer C1.1, C17.1, C20.1, C3.2, C31.1, C32.1, C33.1, C34.1, C36.1, C37.1, FB1.P$1, FB2.P$2, JP3.1, R23.2, R28A.2, R28B.2, R28C.2, R28D.2, R30.2, R4.2, R6.1, U$3.VDD, U1.VSUPPLY, U10.VCC, U13.PS, U13.SDO2, U13.VDD, U13.VDDIO, U15.VIN, U16.VCC, U17.VREF1, U18.BIAS, U4.VCC, U6.VDDIO1, U6.VDDIO2
- net +5V: now also C31.1, C32.1, R14.2, R15.1; no longer C19.1, C23.1, R5.2, R8.1
- net 5V_S: now also R10.2, R5.1, R8.2, R9.2, U6.VDD, U9.A0, U9.A1, U9.A2, U9.VCC; no longer R16.1, R25.2, R26.2, R27.2, U10.VDD, U12.A0, U12.A1, U12.A2, U12.VCC
- net BIAS_REF: now also U2.PB08/EIC/AIN2/SCOM4PAD0/TC4; no longer U6.PB08/EIC/AIN2/SCOM4PAD0/TC4
- net DEC0: now also U9.P15; no longer U12.P15
- net DEC1: now also U9.P13; no longer U12.P13
- net DIR: now also U9.P12; no longer U12.P12
- net EN_28V: now also U2.PA28/EIC; no longer U6.PA28/EIC
- net GND: now also C15.2, C16.2, C17.2, C19.2, C20.1, C21.1, C25.2, C26.2, C28.2, C3.2, C30.2, C4.2, JP1.3, JP1.5, JP2.1, R13.2, R16.2, R6.2, U10.GND, U11.VSS, U13.GND, U13.SYNC, U2.GND1, U2.GND2, U2.GND3, U2.GNDANA, U3.A0, U3.A1, U3.A2, U3.EP, U3.GND, U4.OE, U5.GND, U6.MODE, U6.VSS, U7.CSB3, U7.GNDA, U7.GNDIO, U7.SDO1, U9.EPAD, U9.GND; no longer C20.2, C21.2, C22.2, C3.1, C31.2, C33.2, C34.2, C35.2, C36.2, C37.2, C4.1, C41.2, JP1.1, JP3.3, JP3.5, R2.2, R7.2, R9.2, U$3.VSS, U10.MODE, U10.VSS, U11.A0, U11.A1, U11.A2, U11.EP, U11.GND, U12.EPAD, U13.CSB3, U13.GNDA, U13.GNDIO, U13.SDO1, U15.GND, U15.OE, U16.GND, U17.GND, U18.GND, U18.SYNC, U6.GND1, U6.GND2, U6.GND3, U6.GNDANA
- net I0: now also U9.P17; no longer U12.P17
- net I1: now also U9.P16; no longer U12.P16
- net IMUDR: now also U6.DIN, U7.DRDYM; no longer U10.DIN, U13.DRDYM
- net IMUINT1: now also U6.BIN, U7.INT1; no longer U10.BIN, U13.INT1
- net IMUINT2: now also U6.CIN, U7.INT2; no longer U10.CIN, U13.INT2
- net IMUINT3: now also U6.AIN, U7.INT3; no longer U10.AIN, U13.INT3
- net IMUINT4: now also U6.EIN, U7.INT4; no longer U10.EIN, U13.INT4
- net IMUINT5: now also U6.FIN, U7.INT5; no longer U10.FIN, U13.INT5
- net IOEINT: now also U2.PA17/I2C/EIC/SCOM1PAD1+/TC2, U4.Y; no longer U15.Y, U6.PA17/I2C/EIC/SCOM1PAD1+/TC2
- net I_SENSE: now also U2.PA05/EIC/AIN5/SCOM0PAD1; no longer U6.PA05/EIC/AIN5/SCOM0PAD1
- net LED_CTRL: now also U2.PA09/I2C/EIC/AIN17/SCOM2PAD1+/TC0; no longer U6.PA09/I2C/EIC/AIN17/SCOM2PAD1+/TC0
- net M0: now also U9.P11; no longer U12.P11
- net M1: now also U9.P10; no longer U12.P10
- net MISO: now also U2.PA12/I2C/EIC/SCOM2PAD0+/TC2; no longer U6.PA12/I2C/EIC/SCOM2PAD0+/TC2
- net MOSI: now also U2.PB10/EIC/SCOM4PAD2/TC5; no longer U6.PB10/EIC/SCOM4PAD2/TC5
- net N$1: now also R17.1, U13.RT; no longer R2.1, U18.RT
- net N$10: now also C6.1, C7.1, FB2.P$2, U2.VDDANA; no longer C21.1, C22.1, FB1.P$2, U6.VDDANA
- net N$11: now also C29.1, U13.BOOST2; no longer C16.1, U18.BOOST2
- net N$12: now also C22.1, U13.BOOST1; no longer C15.1, U18.BOOST1
- net N$14: now also C22.2, U13.SW1; no longer C15.2, U18.SW1
- net N$17: now also C29.2, U13.SW2; no longer C16.2, U18.SW2
- net N$19: now also U6.AOUT, U9.P00; no longer U10.AOUT, U12.P00
- net N$2: now also C20.2, U11.VCORE; no longer C4.2, U$3.VCORE
- net N$20: now also R12.1, U13.PG1; no longer R4.1, U18.PG1
- net N$21: now also R14.1, U13.PG2; no longer R5.1, U18.PG2
- net N$22: now also C24.2, R11.2, R13.1, U13.FB1; no longer C17.2, R6.2, R7.1, U18.FB1
- net N$23: now also U6.BOUT, U9.P01; no longer U10.BOUT, U12.P01
- net N$25: now also U4.A, U9.INT; no longer U12.INT, U15.A
- net N$28: now also U6.COUT, U9.P02; no longer U10.COUT, U12.P02
- net N$29: now also U6.DOUT, U9.P03; no longer U10.DOUT, U12.P03
- net N$3: now also C27.1, U13.INTVCC; no longer C12.1, U18.INTVCC
- net N$30: now also U6.EOUT, U9.P04; no longer U10.EOUT, U12.P04
- net N$31: now also U6.FOUT, U9.P05; no longer U10.FOUT, U12.P05
- net N$33: now also R10.1, U10.SDA2, U9.SDA; no longer R27.1, U12.SDA, U17.SDA2
- net N$34: now also R9.1, U10.SCL2, U9.SCL; no longer R25.1, U12.SCL, U17.SCL2
- net N$35: now also C19.1, R8.1, U10.EN, U10.VREF2; no longer C41.1, R26.1, U17.EN, U17.VREF2
- net N$37: now also C31.2, R15.2, R16.1, U13.FB2; no longer C19.2, R8.2, R9.1, U18.FB2
- net N$4: now also C28.1, U13.SS1; no longer C13.1, U18.SS1
- net N$5: now also C5.1, U2.VDDCORE; no longer C27.1, U6.VDDCORE
- net N$6: now also R3.1, U3.OS; no longer R23.1, U11.OS
- net N$7: now also JP2.2, R4.1; no longer JP1.2, R1.1
- net N$8: now also C17.1, U5.VBAT; no longer C5.1, U4.VBAT
- net N$9: now also C30.1, U13.SS2; no longer C14.1, U18.SS2
- net NENBL: now also U9.P07; no longer U12.P07
- net NFAULT: now also U9.P06; no longer U12.P06
- net NSLEEP: now also U9.P14; no longer U12.P14
- net PA27: now also U2.PA27/EIC, U5.!INT!/SQW; no longer U4.!INT!/SQW, U6.PA27/EIC
- net PB02: now also U2.PB02/EIC/AIN10/SCOM5PAD0; no longer U6.PB02/EIC/AIN10/SCOM5PAD0
- net PB03: now also U2.PB03/EIC/AIN11/SCOM5PAD1; no longer U6.PB03/EIC/AIN11/SCOM5PAD1
- net PB22: now also U2.PB22/EIC/SCOM5PAD2; no longer U6.PB22/EIC/SCOM5PAD2
- net PB23: now also U2.PB23/EIC/SCOM5PAD3; no longer U6.PB23/EIC/SCOM5PAD3
- net PI_KILL: now also U2.PA16/I2C/EIC/SCOM1PAD0+/TC2; no longer U6.PA16/I2C/EIC/SCOM1PAD0+/TC2
- net RESET: now also C8.1, JP1.10, R2.1, R4.2, U2.RESET; no longer C10.1, JP3.10, R1.2, R3.1, U6.RESET
- net RX0: now also U2.PA11/EIC/AIN19/SCOM2PAD3+/TC1; no longer U6.PA11/EIC/AIN19/SCOM2PAD3+/TC1
- net RX1: now also U2.PA19/EIC/SCOM1PAD3+/TC3; no longer U6.PA19/EIC/SCOM1PAD3+/TC3
- net RX2: now also U2.PA21/EIC/SCOM5PAD3+; no longer U6.PA21/EIC/SCOM5PAD3+
- net SCK: now also U2.PB11/EIC/SCOM4PAD3/TC5; no longer U6.PB11/EIC/SCOM4PAD3/TC5
- net SCL: now also R7C.1, U1.SCL0, U10.SCL1, U12.SCL, U2.PA23/I2C/EIC/SCOM5PAD1+/TC4, U3.SCL, U5.SCL, U7.SCX; no longer R28C.1, U$3.SCL, U1.SCL, U13.SCX, U16.SCL0, U17.SCL1, U4.SCL, U6.PA23/I2C/EIC/SCOM5PAD1+/TC4
- net SCL_BUFF: now also R7B.1, U1.SCL1; no longer R28B.1, U16.SCL1
- net SDA: now also R7D.1, U1.SDA0, U10.SDA1, U12.SDA, U2.PA22/I2C/EIC/SCOM5PAD0+/TC4, U3.SDA, U5.SDA, U7.SDX; no longer R28D.1, U$3.SDA, U1.SDA, U13.SDX, U16.SDA0, U17.SDA1, U4.SDA, U6.PA22/I2C/EIC/SCOM5PAD0+/TC4
- net SDA_BUFF: now also R7A.1, U1.SDA1; no longer R28A.1, U16.SDA1
- net STEPFREQ: now also U2.PA08/I2C/AIN16/SCOM2PAD0+/TC0; no longer U6.PA08/I2C/AIN16/SCOM2PAD0+/TC0
- net SWDCLK: now also JP1.4, R1.1, U2.PA30/EIC/SCOM1PAD2/SWDCLK; no longer JP3.4, R30.1, U6.PA30/EIC/SCOM1PAD2/SWDCLK
- net SWDIO: now also JP1.2, U2.PA31/EIC/SCOM1PAD3/SWDIO; no longer JP3.2, U6.PA31/EIC/SCOM1PAD3/SWDIO
- net SYNC: now also U2.PA15/XOUT/EIC/SCOM2PAD3+/TC3; no longer U6.PA15/XOUT/EIC/SCOM2PAD3+/TC3
- net TX0: now also U2.PA10/EIC/AIN18/SCOM2PAD2+/TC1; no longer U6.PA10/EIC/AIN18/SCOM2PAD2+/TC1
- net TX1: now also U2.PA18/EIC/SCOM1PAD2+/TC3; no longer U6.PA18/EIC/SCOM1PAD2+/TC3
- net TX2: now also U2.PA20/EIC/SCOM5PAD2+; no longer U6.PA20/EIC/SCOM5PAD2+
- net USB_D_N: now also U2.PA24/EIC/SCOM3PAD2+/TC5; no longer U6.PA24/EIC/SCOM3PAD2+/TC5
- net USB_D_P: now also U2.PA25/EIC/SCOM3PAD3+/TC5; no longer U6.PA25/EIC/SCOM3PAD3+/TC5
- net VDD: now also C23.1, C26.1, U13.EN1, U13.EN2, U13.VIN1, U13.VIN2; no longer C11.1, C6.1, U18.EN1, U18.EN2, U18.VIN1, U18.VIN2
- net VREFA: now also C1.1, FB1.P$1, U2.PA03/EIC/REF/AI/VREFA; no longer C35.1, FB2.P$1, U6.PA03/EIC/REF/AI/VREFA
- net V_SENSE: now also R5.2, R6.1, U2.PA02/EIC/AIN; no longer R16.2, R17.1, U6.PA02/EIC/AIN
- net XIN32: now also C10.1, U2.PA00/XIN32/EIC/SCOM1PAD0; no longer C7.1, U6.PA00/XIN32/EIC/SCOM1PAD0
- net XOUT32: now also C11.1, U2.PA01/XOUT32/EIC/SCOM1PAD1; no longer C8.1, U6.PA01/XOUT32/EIC/SCOM1PAD1
Other:
- moved on the sheet: B1, C1, C10, C11, C12, C13, C14, C15, C16, C17, C18, C19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
