File: STAR/Eagle/STARduino/starduino.brd (EAGLE design)
At the start: 59.7 x 38.2 mm, 76 parts, among them J1 J30J-25, Q2 BSS8402DW, U1 SSCMNNN015PA2A3, U10 MC14504BDTG, U11 MAX31725MTA+, U12 TCA9535_RTW_24, U13 BMX055, U15 MC74VHC1GT125, U16 PCA9515A, U17 PCA9306DCT, U18 LT8616, U4 DS3231MZ+, U6 ATSAMD21G18, U8 ADXL375BCCZ

Commit message: screws
Parts:
- moved B1 0.13 mm to (39.7, 32.0)
Connections:
- removed net D: J1.10
- removed net N$27: J1.11
- removed net N$32: J1.12
- removed net N$36: J1.13
Changed lines of the file:
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@@
 <hole x="48.768" y="36.1315" drill="2.1"/>
 <hole x="57.4675" y="2.0955" drill="2.1"/>
-<hole x="2.7305" y="2.0955" drill="2.1"/>
+<hole x="2.7305" y="2.032" drill="2.1"/>
 <wire x1="0" y1="1.27" x2="0" y2="36.83" width="0" layer="20"/>
 <wire x1="1.27" y1="38.1" x2="58.9915" y2="38.1" width="0" layer="20"/>
+<circle x="7.874" y="32.512" radius="1.9" width="0.4064" layer="51"/>
+<circle x="2.7305" y="2.032" radius="1.9" width="0.4064" layer="51"/>
+<circle x="48.768" y="36.1315" radius="1.9" width="0.4064" layer="51"/>
+<circle x="57.4675" y="2.0955" radius="1.9" width="0.4064" layer="51"/>
 </plain>
 <attributes>
@@
 <element name="C37" library="resistor" package="C0603" value="100nF" x="49.911" y="5.87375" rot="R90"/>
 <element name="U4" library="NR_IC" package="SOIC-8" value="DS3231MZ+" x="24.3205" y="23.9395"/>
-<element name="B1" library="NR_connectors" package="CR1025" value="CR1025" x="39.671625" y="32.115125"/>
+<element name="B1" library="NR_connectors" package="CR1025" value="CR1025" x="39.671625" y="31.988125"/>
 <element name="C9" library="resistor" package="C0603" value="100nF" x="21.129625" y="31.90875" rot="R270"/>
 <element name="C5" library="resistor" package="C0603" value="1nF" x="24.971375" y="29.24175" rot="R180"/>
@@
 <contactref element="B1" pad="1"/>
 <contactref element="B1" pad="2"/>
-<wire x1="31.976625" y1="32.115125" x2="31.976625" y2="34.897625" width="0.381" layer="1"/>
+<wire x1="31.976625" y1="31.988125" x2="31.976625" y2="34.897625" width="0.381" layer="1"/>
 <wire x1="31.976625" y1="34.897625" x2="33.9725" y2="36.8935" width="0.381" layer="1"/>
 <wire x1="33.9725" y1="36.8935" x2="44.577" y2="36.8935" width="0.381" layer="1"/>
 <wire x1="44.577" y1="36.8935" x2="47.244" y2="34.2265" width="0.381" layer="1"/>
 <wire x1="47.244" y1="34.2265" x2="47.244" y2="32.23775" width="0.381" layer="1"/>
-<wire x1="47.244" y1="32.23775" x2="47.366625" y2="32.115125" width="0.381" layer="1"/>
+<wire x1="47.244" y1="32.23775" x2="47.366625" y2="31.988125" width="0.381" layer="1"/>
 <wire x1="25.821375" y1="29.24175" x2="24.9555" y2="28.375875" width="0.381" layer="1"/>
 <wire x1="24.9555" y1="28.375875" x2="24.9555" y2="26.7395" width="0.381" layer="1"/>
@@
 <wire x1="32.385" y1="31.9405" x2="32.512" y2="32.0675" width="0.381" layer="1"/>
 <wire x1="32.512" y1="32.0675" x2="32.02425" y2="32.0675" width="0.381" layer="1"/>
-<wire x1="32.02425" y1="32.0675" x2="31.976625" y2="32.115125" width="0.381" layer="1"/>
+<wire x1="32.02425" y1="32.0675" x2="31.976625" y2="31.988125" width="0.381" layer="1"/>
 </signal>
 <signal name="TX0">
@@
 <wire x1="53.086" y1="13.04925" x2="55.84825" y2="15.8115" width="0.3048" layer="16"/>
 </signal>
-<signal name="D">
-<contactref element="J1" pad="10"/>
-</signal>
 <signal name="SD_STAR">
 <contactref element="J1" pad="9"/>
 </signal>
-<signal name="N$27">
-<contactref element="J1" pad="11"/>
-</signal>
-<signal name="N$32">
-<contactref element="J1" pad="12"/>
-</signal>
-<signal name="N$36">
-<contactref element="J1" pad="13"/>
-</signal>
 <signal name="N$2">

Commit message: external kill
Parts:
- removed Q2: BSS8402DW, transistor-fet:SC70
- removed R13: 100k, resistor:R0603
- removed R15: 191k, resistor:R0603
Connections:
- removed net DEBUG_5V: Q2.3
- removed net EXTERNAL_KILL: Q2.2, R13.1, U16.P$5, U6.22
- removed net N$38: Q2.5, Q2.6, R15.2
- net +5V: no longer Q2.4, R15.1
- net GND: no longer Q2.1, R13.2
Routing:
- net EXTERNAL_KILL: track 38.1 -> 0.00 mm, vias 2 -> 0
- net +5V: track 117.9 -> 110.2 mm
- net GND: track 256.4 -> 253.3 mm
- net N$38: track 2.84 -> 0.00 mm
Changed lines of the file:
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@@
 <element name="U17" library="MotorDriver" package="SSOP8" value="PCA9306DCT" x="39.068375" y="18.89125" rot="R270"/>
 <element name="U15" library="CM_IC" package="SC-70-5" value="MC74VHC1GT125" x="37.830125" y="15.128875" rot="R90"/>
-<element name="R15" library="resistor" package="R0603" value="191k" x="32.3215" y="3.063875" rot="R90"/>
-<element name="R13" library="resistor" package="R0603" value="100k" x="31.861125" y="6.1595" rot="R90"/>
 <element name="JP1" library="CM_passives" package="1X02" value="" x="1.857375" y="36.35375"/>
 <element name="U$2" library="images" package="SSL_SILK_.3IN" value="SSL.3IN_SILK" x="12.303125" y="11.90625" rot="MR0"/>
 <element name="U$1" library="images" package="STAR_.3IN" value="STAR" x="25.161875" y="12.144375" rot="MR0"/>
 <element name="R28" library="SparkFun-Passives" package="0603-ARV" value="4.7k" x="20.16125" y="8.47725"/>
-<element name="Q2" library="transistor-fet" package="SC70" value="BSS8402DW" x="30.0355" y="1.651" rot="R270"/>
 <element name="U16" library="CM_IC" package="TSSOP8" value="PCA9515A" x="25.05075" y="4.238625" rot="R270"/>
 <element name="JP3" library="pinhead" package="2X05" value="" x="3.048" y="28.2575" rot="R90"/>
@@
 <contactref element="U10" pad="13"/>
 <contactref element="U12" pad="25"/>
-<contactref element="R13" pad="2"/>
 <contactref element="U15" pad="3"/>
 <contactref element="U15" pad="1"/>
 <contactref element="JP1" pad="1"/>
-<contactref element="Q2" pad="1"/>
 <contactref element="C41" pad="2"/>
 <contactref element="U16" pad="P$4"/>
@@
 <via x="32.5755" y="16.0655" extent="1-16" drill="0.6"/>
 <via x="32.5755" y="13.843" extent="1-16" drill="0.6"/>
-<wire x1="31.861125" y1="7.0095" x2="32.171375" y2="7.31975" width="0.2032" layer="1"/>
 <wire x1="32.171375" y1="7.31975" x2="32.171375" y2="9.604375" width="0.2032" layer="1"/>
 <wire x1="29.1465" y1="8.69225" x2="28.798625" y2="9.040125" width="0.2032" layer="1"/>
@@
 <vertex x="0" y="-1.27"/>
 </polygon>
-<wire x1="29.1355" y1="2.351" x2="26.478" y2="2.351" width="0.2032" layer="1"/>
 <via x="26.416" y="2.413" extent="1-16" drill="0.5238"/>
 <wire x1="26.416" y1="2.413" x2="26.416" y2="5.7785" width="0.2032" layer="16"/>
@@
 </signal>
 <signal name="+5V">
-<contactref element="R15" pad="1"/>
-<contactref element="Q2" pad="4"/>
 <contactref element="L2" pad="P$2"/>
 <contactref element="R8" pad="1"/>
@@
 <wire x1="17.184" y1="26.9875" x2="15.3815" y2="25.185" width="1.016" layer="1"/>
 <wire x1="15.3815" y1="25.185" x2="12.2555" y2="25.185" width="1.016" layer="1"/>
-<wire x1="37.17925" y1="3.14325" x2="36.8935" y2="2.794" width="1.016" layer="1"/>
-<wire x1="36.8935" y1="2.794" x2="32.901625" y2="2.794" width="0.762" layer="1"/>
-<wire x1="32.901625" y1="2.794" x2="32.3215" y2="2.213875" width="0.762" layer="1"/>
-<wire x1="32.3215" y1="2.213875" x2="32.3215" y2="1.27" width="0.508" layer="1"/>
-<wire x1="32.3215" y1="1.27" x2="32.0675" y2="1.016" width="0.508" layer="1"/>
-<wire x1="32.0675" y1="1.016" x2="31.0005" y2="1.016" width="0.508" layer="1"/>
-<wire x1="31.0005" y1="1.016" x2="30.9355" y2="0.951" width="0.508" layer="1"/>
 <wire x1="9.525" y1="25.185" x2="9.525" y2="23.8125" width="1.016" layer="1"/>
 <wire x1="9.525" y1="23.8125" x2="12.2555" y2="21.082" width="1.016" layer="1"/>
@@
 <contactref element="U6" pad="24"/>
 </signal>
-<signal name="EXTERNAL_KILL">
-<contactref element="R13" pad="1"/>
-<contactref element="U6" pad="22"/>
-<contactref element="Q2" pad="2"/>
-<contactref element="U16" pad="P$5"/>
-<wire x1="31.861125" y1="5.3095" x2="31.861125" y2="5.000625" width="0.381" layer="1"/>
-<wire x1="31.861125" y1="5.000625" x2="30.0355" y2="3.175" width="0.381" layer="1"/>
-<wire x1="30.0355" y1="3.175" x2="27.449625" y2="3.175" width="0.381" layer="1"/>
-<wire x1="27.449625" y1="3.175" x2="27.42575" y2="3.151125" width="0.381" layer="1"/>
-<via x="30.607" y="16.7005" extent="1-16" drill="0.5238"/>
-<wire x1="30.607" y1="17.272" x2="30.607" y2="16.7005" width="0.3048" layer="1"/>
-<wire x1="30.607" y1="16.7005" x2="30.607" y2="14.478" width="0.3048" layer="16"/>
-<wire x1="35.1409" y1="18.4785" x2="34.0995" y2="18.4785" width="0.3048" layer="1"/>
-<wire x1="34.0995" y1="18.4785" x2="34.036" y2="18.542" width="0.3048" layer="1"/>
-<wire x1="34.036" y1="18.542" x2="34.036" y2="18.923" width="0.3048" layer="1"/>
-<wire x1="34.036" y1="18.923" x2="33.7185" y2="19.2405" width="0.3048" layer="1"/>
-<wire x1="33.7185" y1="19.2405" x2="31.496" y2="19.2405" width="0.3048" layer="1"/>
-<wire x1="31.496" y1="19.2405" x2="30.734" y2="18.4785" width="0.3048" layer="1"/>
-<wire x1="30.734" y1="18.4785" x2="30.734" y2="17.399" width="0.3048" layer="1"/>
-<wire x1="30.734" y1="17.399" x2="30.607" y2="17.272" width="0.3048" layer="1"/>
-<wire x1="35.1409" y1="18.4785" x2="35.1663" y2="18.4531" width="0.3048" layer="1"/>
-<wire x1="31.861125" y1="5.3095" x2="36.234" y2="5.3095" width="0.3048" layer="1"/>
-<wire x1="36.234" y1="5.3095" x2="36.2585" y2="5.334" width="0.3048" layer="1"/>
-<via x="36.2585" y="5.334" extent="1-16" drill="0.6"/>
-<wire x1="36.2585" y1="5.334" x2="36.2585" y2="5.9055" width="0.3048" layer="16"/>
-<wire x1="36.2585" y1="5.9055" x2="34.2265" y2="7.9375" width="0.3048" layer="16"/>
-<wire x1="34.2265" y1="7.9375" x2="34.2265" y2="12.2555" width="0.3048" layer="16"/>
-<wire x1="34.2265" y1="12.2555" x2="33.5915" y2="12.8905" width="0.3048" layer="16"/>
-<wire x1="33.5915" y1="12.8905" x2="32.258" y2="12.8905" width="0.3048" layer="16"/>
-<wire x1="32.258" y1="12.8905" x2="30.607" y2="14.478" width="0.3048" layer="16"/>
-<wire x1="26.035" y1="1.5875" x2="25.527" y2="2.0955" width="0.381" layer="1"/>
-<wire x1="25.527" y1="2.0955" x2="25.527" y2="2.667" width="0.381" layer="1"/>
-<wire x1="25.527" y1="2.667" x2="26.0985" y2="3.2385" width="0.381" layer="1"/>
-<wire x1="26.0985" y1="3.2385" x2="27.338375" y2="3.2385" width="0.381" layer="1"/>
-<wire x1="27.338375" y1="3.2385" x2="27.42575" y2="3.151125" width="0.381" layer="1"/>
-<wire x1="26.035" y1="1.5875" x2="29.072" y2="1.5875" width="0.381" layer="1"/>
-<wire x1="29.072" y1="1.5875" x2="29.1355" y2="1.651" width="0.381" layer="1"/>
-</signal>
 <signal name="PI_KILL">
 <contactref element="U6" pad="25"/>
 </signal>
-<signal name="N$38">
-<contactref element="R15" pad="2"/>
-<contactref element="Q2" pad="6"/>
-<contactref element="Q2" pad="5"/>
-<wire x1="30.9355" y1="1.651" x2="30.9355" y2="2.351" width="0.381" layer="1"/>
-<wire x1="30.9355" y1="2.351" x2="30.9355" y2="2.527875" width="0.381" layer="1"/>
-<wire x1="30.9355" y1="2.527875" x2="32.3215" y2="3.913875" width="0.381" layer="1"/>
-</signal>
-<signal name="DEBUG_5V">
-<contactref element="Q2" pad="3"/>
-</signal>
 <signal name="SCL_BUFF">

Commit message: moved stuff on STARduino
Parts:
- moved R9 5.08 mm to (8.83, 29.8), turned to 90 degrees
- moved C12 4.18 mm to (8.38, 32.9)
- moved R2 3.86 mm to (6.99, 32.1)
- moved R8 3.74 mm to (13.1, 25.1)
- moved C19 2.54 mm to (14.6, 25.1)
- moved C14 1.12 mm to (11.7, 25.3)
- moved C10 0.63 mm to (8.00, 20.4)
Routing:
- net GND: track 253.3 -> 231.6 mm, vias 41 -> 37
- net +5V: track 110.2 -> 103.5 mm
- net N$1: track 14.4 -> 11.0 mm
- net RESET: track 48.4 -> 45.6 mm
- net N$37: track 16.4 -> 13.8 mm
- net N$3: track 5.42 -> 2.83 mm
- net N$9: track 1.54 -> 2.65 mm
