File: STAR/Eagle/BiasGenerator/bias_generator.sch (EAGLE design)
At the start: 24 parts, among them J1 J30J-9J30, T1 750311838, U1 LT8300, U2 LT8330

Commit message: bias gen board
Connections:
- new net G: J1.3
- new net N$10: J1.9
- net +50V: now also J1.1, J1.2; no longer J1.3, J1.4
- net GND: now also J1.6; no longer J1.1, J1.2
- net VCC: now also J1.4; no longer J1.6
Changed lines of the file:
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@@
+</segment>
+<segment>
+<pinref part="J1" gate="G$1" pin="4"/>
+<wire x1="233.68" y1="68.58" x2="231.14" y2="68.58" width="0.1524" layer="91"/>
+<label x="231.14" y="68.58" size="1.016" layer="95" rot="R180" xref="yes"/>
+</segment>
+</net>
+<net name="GND" class="0">
+<segment>
+<pinref part="C1" gate="G$1" pin="2"/>
+<pinref part="GND2" gate="1" pin="GND"/>
+</segment>
+<segment>
+<pinref part="C2" gate="G$1" pin="2"/>
+<pinref part="GND3" gate="1" pin="GND"/>
+</segment>
+<segment>
+<pinref part="U1" gate="G$1" pin="GND"/>
+<pinref part="GND4" gate="1" pin="GND"/>
+</segment>
+<segment>
+<pinref part="T1" gate="G$1" pin="S2A"/>
+<pinref part="GND5" gate="1" pin="GND"/>
+<wire x1="139.7" y1="172.72" x2="144.78" y2="172.72" width="0.1524" layer="91"/>
+</segment>
+<segment>
+<pinref part="C3" gate="G$1" pin="2"/>
+<pinref part="GND6" gate="1" pin="GND"/>
+</segment>
+<segment>
+<pinref part="C4" gate="G$1" pin="2"/>
+<pinref part="GND7" gate="1" pin="GND"/>
+</segment>
+<segment>
+<pinref part="C5" gate="G$1" pin="2"/>
+<pinref part="GND8" gate="1" pin="GND"/>
+</segment>
+<segment>
+<pinref part="GND1" gate="1" pin="GND"/>
+<wire x1="73.66" y1="50.8" x2="73.66" y2="58.42" width="0.1524" layer="91"/>
+<pinref part="U2" gate="G$1" pin="GND"/>
+</segment>
+<segment>
+<pinref part="R5" gate="G$1" pin="1"/>
+<pinref part="GND9" gate="1" pin="GND"/>
+</segment>
+<segment>
+<pinref part="GND10" gate="1" pin="GND"/>
+<pinref part="C7" gate="G$1" pin="2"/>
+</segment>
+<segment>
+<pinref part="R6" gate="G$1" pin="1"/>
+<pinref part="GND11" gate="1" pin="GND"/>
+</segment>
+<segment>
+<wire x1="218.44" y1="152.4" x2="218.44" y2="147.32" width="0.1524" layer="91"/>
+<pinref part="GND12" gate="1" pin="GND"/>
+<pinref part="R8" gate="G$1" pin="1"/>
+</segment>
+<segment>
+<pinref part="J1" gate="G$1" pin="7"/>
+<wire x1="243.84" y1="76.2" x2="246.38" y2="76.2" width="0.1524" layer="91"/>
+<label x="246.38" y="76.2" size="1.016" layer="95" xref="yes"/>
+</segment>
+<segment>
+<wire x1="243.586" y1="71.12" x2="246.634" y2="71.12" width="0.1524" layer="91"/>
+<label x="246.38" y="71.12" size="1.016" layer="95" xref="yes"/>
 </segment>
 <segment>
@@
 <wire x1="243.84" y1="81.28" x2="246.38" y2="81.28" width="0.1524" layer="91"/>
 <label x="246.38" y="81.28" size="1.016" layer="95" xref="yes"/>
-</segment>
-</net>
-<net name="GND" class="0">
-<segment>
-<pinref part="C1" gate="G$1" pin="2"/>
-<pinref part="GND2" gate="1" pin="GND"/>
-</segment>
-<segment>
-<pinref part="C2" gate="G$1" pin="2"/>
-<pinref part="GND3" gate="1" pin="GND"/>
-</segment>
-<segment>
-<pinref part="U1" gate="G$1" pin="GND"/>
-<pinref part="GND4" gate="1" pin="GND"/>
-</segment>
-<segment>
-<pinref part="T1" gate="G$1" pin="S2A"/>
-<pinref part="GND5" gate="1" pin="GND"/>
-<wire x1="139.7" y1="172.72" x2="144.78" y2="172.72" width="0.1524" layer="91"/>
-</segment>
-<segment>
-<pinref part="C3" gate="G$1" pin="2"/>
-<pinref part="GND6" gate="1" pin="GND"/>
-</segment>
-<segment>
-<pinref part="C4" gate="G$1" pin="2"/>
-<pinref part="GND7" gate="1" pin="GND"/>
-</segment>
-<segment>
-<pinref part="C5" gate="G$1" pin="2"/>
-<pinref part="GND8" gate="1" pin="GND"/>
-</segment>
-<segment>
-<pinref part="GND1" gate="1" pin="GND"/>
-<wire x1="73.66" y1="50.8" x2="73.66" y2="58.42" width="0.1524" layer="91"/>
-<pinref part="U2" gate="G$1" pin="GND"/>
-</segment>
-<segment>
-<pinref part="R5" gate="G$1" pin="1"/>
-<pinref part="GND9" gate="1" pin="GND"/>
-</segment>
-<segment>
-<pinref part="GND10" gate="1" pin="GND"/>
-<pinref part="C7" gate="G$1" pin="2"/>
-</segment>
-<segment>
-<pinref part="R6" gate="G$1" pin="1"/>
-<pinref part="GND11" gate="1" pin="GND"/>
-</segment>
-<segment>
-<wire x1="218.44" y1="152.4" x2="218.44" y2="147.32" width="0.1524" layer="91"/>
-<pinref part="GND12" gate="1" pin="GND"/>
-<pinref part="R8" gate="G$1" pin="1"/>
-</segment>
-<segment>
-<pinref part="J1" gate="G$1" pin="1"/>
-<wire x1="233.68" y1="83.82" x2="231.14" y2="83.82" width="0.1524" layer="91"/>
-<label x="231.14" y="83.82" size="1.016" layer="95" rot="R180" xref="yes"/>
-</segment>
-<segment>
-<pinref part="J1" gate="G$1" pin="2"/>
-<wire x1="233.68" y1="78.74" x2="231.14" y2="78.74" width="0.1524" layer="91"/>
-<label x="231.14" y="78.74" size="1.016" layer="95" rot="R180" xref="yes"/>
-</segment>
-<segment>
-<pinref part="J1" gate="G$1" pin="7"/>
-<wire x1="243.84" y1="76.2" x2="246.38" y2="76.2" width="0.1524" layer="91"/>
-<label x="246.38" y="76.2" size="1.016" layer="95" xref="yes"/>
 </segment>
 </net>
@@
 </segment>
 <segment>
-<pinref part="J1" gate="G$1" pin="3"/>
-<wire x1="233.68" y1="73.66" x2="231.14" y2="73.66" width="0.1524" layer="91"/>
-<label x="231.14" y="73.66" size="1.016" layer="95" rot="R180" xref="yes"/>
-</segment>
-<segment>
-<pinref part="J1" gate="G$1" pin="4"/>
-<wire x1="233.68" y1="68.58" x2="231.14" y2="68.58" width="0.1524" layer="91"/>
-<label x="231.14" y="68.58" size="1.016" layer="95" rot="R180" xref="yes"/>
+<pinref part="J1" gate="G$1" pin="1"/>
+<wire x1="233.68" y1="83.82" x2="231.14" y2="83.82" width="0.1524" layer="91"/>
+<label x="231.14" y="83.82" size="1.016" layer="95" rot="R180" xref="yes"/>
+</segment>
+<segment>
+<pinref part="J1" gate="G$1" pin="2"/>
+<wire x1="233.68" y1="78.74" x2="231.14" y2="78.74" width="0.1524" layer="91"/>
+<label x="231.14" y="78.74" size="1.016" layer="95" rot="R180" xref="yes"/>
 </segment>
 </net>
@@
 </segment>
 </net>
+<net name="N$10" class="0">
+<segment>
+<pinref part="J1" gate="G$1" pin="9"/>
+<wire x1="243.84" y1="66.04" x2="246.38" y2="66.04" width="0.1524" layer="91"/>
+<label x="246.38" y="66.04" size="1.016" layer="95" xref="yes"/>
+</segment>
+</net>
+<net name="G" class="0">
+<segment>
+<pinref part="J1" gate="G$1" pin="3"/>
+<wire x1="233.68" y1="73.66" x2="231.14" y2="73.66" width="0.1524" layer="91"/>
+<label x="231.14" y="73.66" size="1.016" layer="95" rot="R180" xref="yes"/>
+</segment>
+</net>

Commit message: screws
Connections:
- removed net G: J1.3
Changed lines of the file:
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@@
 <pinref part="J1" gate="G$1" pin="9"/>
 <wire x1="243.84" y1="66.04" x2="246.38" y2="66.04" width="0.1524" layer="91"/>
-<label x="246.38" y="66.04" size="1.016" layer="95" xref="yes"/>
 </segment>
 </net>
-<net name="G" class="0">
-<segment>
-<pinref part="J1" gate="G$1" pin="3"/>
-<wire x1="233.68" y1="73.66" x2="231.14" y2="73.66" width="0.1524" layer="91"/>
-<label x="231.14" y="73.66" size="1.016" layer="95" rot="R180" xref="yes"/>
-</segment>
-</net>

Commit message: misc board stuff
Parts:
- C4: value 1uF -> 10uF; device AR_passives:CAPACITORC0603 -> AR_passives:CAPACITOR2-J-LEAD
- C7: value 10uF -> 1uF; device AR_passives:CAPACITOR2-J-LEAD -> AR_passives:CAPACITORC0603
- D1: value BAV20W -> MMSZ5266BT1G; device AR_diode:SCHOTTKYSOD323 -> AR_diode:ZENERSOD123
- D2: value MMSZ5266BT1G -> BAV20W; device AR_diode:ZENERSOD123 -> AR_diode:SCHOTTKYSOD323
- R1: value 407k -> 47k; device resistor:R-US_R0603 -> resistor:R-US_R2512
- R2: value 1k -> 407k
- R3: value 1M -> 1k
- R4: value 1M -> 3k; device resistor:R-US_R0603 -> resistor:R-US_R2512
- R5: value 1M -> 1.5k; device resistor:R-US_R0603 -> resistor:R-US_R2512
- R6: value 1.5k -> 1M; device resistor:R-US_R2512 -> resistor:R-US_R0603
- R7: value 47k -> 1M; device resistor:R-US_R2512 -> resistor:R-US_R0603
- R8: value 3k -> 1M; device resistor:R-US_R2512 -> resistor:R-US_R0603
Connections:
- net +20V: now also C5.1; no longer C4.1
- net +50V: now also C4.1, R1.2, R5.2; no longer C7.1, R3.2, R7.2
- net GND: now also R4.1; no longer R6.1
- net N$11: now also R7.1, R8.2; no longer R4.1, R5.2
- net N$2: now also R2.1; no longer R1.1
- net N$3: now also R2.2, R3.1; no longer R1.2, R2.1
- net N$4: now also D2.A, R3.2; no longer D1.A, R2.2
- net N$6: now also C7.1; no longer C5.1
- net N$9: now also R6.1, R7.2; no longer R3.1, R4.2
- net VCC: now also D1.A; no longer D2.A
- net V_DIVIDE: now also R1.1, R4.2; no longer R7.1, R8.2
Other:
- moved on the sheet: C4, C5, C7, R1, R2, R3, R4, R5, R6, R7, R8
