File: STAR/Eagle/Datalogger/datalogger.brd (EAGLE design)
At the start: 26.4 x 55.9 mm, 7 parts, among them J1 J30J-25

Commit message: datalogger 2.1
Connections:
- removed net B: J1.18
- removed net H: J1.19
- net GND: now also J1.18
- net MISO_STAR: now also J1.13, U$1.DAT0; no longer J1.25, U$1.CMD
- net MOSI_STAR: now also J1.25, U$1.CMD; no longer J1.13, U$1.DAT0
Routing:
- net MOSI_STAR: track 16.4 -> 13.5 mm
- net MISO_STAR: track 13.5 -> 16.4 mm
Other:
- board text added: "3.2018"
- board text added: "v. 2.1"
- board text removed: "1.2018"
- board text removed: "v. 2"
Changed lines of the file:
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@@
 <wire x1="12.192" y1="40.64" x2="-11.684" y2="40.64" width="0" layer="20"/>
 <text x="-12.065" y="23.1775" size="1.016" layer="21" font="vector">Datalogger</text>
-<text x="-12.065" y="21.9075" size="1.016" layer="21" font="vector">v. 2</text>
-<text x="-12.065" y="20.32" size="1.016" layer="21" font="vector">1.2018</text>
+<text x="-12.065" y="21.9075" size="1.016" layer="21" font="vector">v. 2.1</text>
+<text x="-12.065" y="20.32" size="1.016" layer="21" font="vector">3.2018</text>
 <text x="8.636" y="20.447" size="1.016" layer="21" font="vector">1</text>
 <text x="5.715" y="29.845" size="1.016" layer="21" font="vector">2</text>
@@
 <vertex x="16.51" y="41.91"/>
 </polygon>
+<contactref element="J1" pad="18"/>
 </signal>
 <signal name="+3V3">
@@
 <wire x1="1.485" y1="29.4885" x2="3.81" y2="31.75" width="0.254" layer="1"/>
 </signal>
-<signal name="MISO_STAR">
+<signal name="MOSI_STAR">
 <contactref element="U$1" pad="CMD"/>
 <contactref element="J1" pad="25"/>
@@
 <wire x1="4.445" y1="33.3375" x2="4.445" y2="33.02" width="0.254" layer="1"/>
 </signal>
-<signal name="MOSI_STAR">
+<signal name="MISO_STAR">
 <contactref element="U$1" pad="DAT0"/>
 <contactref element="J1" pad="13"/>
@@
 <wire x1="11.557" y1="17.907" x2="12.065" y2="18.415" width="0.254" layer="1"/>
 </signal>
-<signal name="B">
-<contactref element="J1" pad="18"/>
-</signal>
-<signal name="H">
-<contactref element="J1" pad="19"/>
-</signal>
 <signal name="N$10">
