File: STAR/Eagle/Datalogger/datalogger.brd (EAGLE design)
At the start: 26.4 x 55.9 mm, 6 parts, among them J1 J30J-25

Commit message: Datalogger v4
Parts:
- added C1, C3, C6, C7, C9: 0.1uF, resistor:C0603
- added C10, C2, C4, C5, C8: 10nF, resistor:C0603
- moved R2 16.0 mm to (3.62, 38.4), turned to 90 degrees
- moved U$1 0.60 mm to (-8.13, 25.4)
- renumbered U$4 to GND1
Connections:
- removed net +5V: J1.1, J1.19, R2.2, U$2.VCC1, U$2.VCC2, U$3.VCC1, U$3.VCC2
- removed net N$1: J1.14
- removed net N$2: J1.15
- removed net N$4: J1.6
- removed net N$5: J1.7
- removed net N$6: J1.8
- removed net N$7: J1.9
- removed net N$8: J1.10
- removed net SD_STAR: J1.24, R2.1, U$1.CD
- new net +5V1: C3.1, C4.1, J1.4, U$2.VCC1
- new net +5V2: C5.1, C6.1, J1.22, U$2.VCC2
- new net +5V3: C10.1, C9.1, J1.17, U$3.VCC1
- new net +5V4: C7.1, C8.1, J1.19, U$3.VCC2
- new net CS_STAR: R2.1, U$1.CD
- new net GND1: C3.2, C4.2, J1.3, J1.5, U$2.GND1
- new net GND2: C5.2, C6.2, J1.8, J1.9, U$2.GND2
- new net GND3: C10.2, C9.2, J1.16, J1.18, U$3.GND1
- new net GND4: C7.2, C8.2, J1.6, J1.7, U$3.GND2
- net +3V3: now also C1.1, C2.1, J1.13, R2.2; no longer J1.12
- net DATA1_N: now also U$2.DATA+1; no longer U$2.DATA-1
- net DATA1_P: now also J1.1, U$2.DATA-1; no longer J1.4, U$2.DATA+1
- net DATA2_N: now also U$2.DATA+2; no longer U$2.DATA-2
- net DATA2_P: now also J1.25, U$2.DATA-2; no longer J1.22, U$2.DATA+2
- net DATA3_N: now also J1.15, U$3.DATA+1; no longer J1.16, U$3.DATA-1
- net DATA3_P: now also J1.14, U$3.DATA-1; no longer J1.17, U$3.DATA+1
- net DATA4_N: now also J1.20, U$3.DATA+2; no longer J1.21, U$3.DATA-2
- net DATA4_P: now also J1.21, U$3.DATA-2; no longer J1.20, U$3.DATA+2
- net GND: now also C1.2, C2.2, J1.11; no longer J1.18, U$2.GND1, U$2.GND2, U$3.GND1, U$3.GND2
- net MISO_STAR: now also J1.12; no longer J1.13
- net MOSI_STAR: now also J1.24; no longer J1.25
- net SCK_STAR: now also J1.10; no longer J1.11
Routing:
- net +5V2: track 0.00 -> 62.2 mm
- net +5V: track 61.0 -> 0.00 mm
- net +5V1: track 0.00 -> 33.0 mm
- net SD_STAR: track 26.7 -> 0.00 mm
- net GND: track 0.00 -> 22.9 mm, vias 14 -> 6
- net +5V4: track 0.00 -> 21.5 mm
- net DATA2_P: track 51.9 -> 69.9 mm
- net DATA2_N: track 52.0 -> 69.9 mm
- net CS_STAR: track 0.00 -> 15.6 mm, vias 0 -> 2
- net +3V3: track 18.3 -> 33.7 mm, vias 0 -> 1
- net +5V3: track 0.00 -> 15.1 mm
- net GND4: track 0.00 -> 14.6 mm, vias 0 -> 7
- net GND2: track 0.00 -> 9.78 mm, vias 0 -> 12
- net MOSI_STAR: track 13.5 -> 17.1 mm
- net DATA4_N: track 31.8 -> 29.5 mm
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- added copper zone on layer 1, net GND1
- added copper zone on layer 16, net GND1
- added copper zone on layer 1, net GND2
- added copper zone on layer 16, net GND2
- added copper zone on layer 1, net GND3
- added copper zone on layer 16, net GND3
- added copper zone on layer 1, net GND4
- added copper zone on layer 16, net GND4
Other:
- board size 26.4 x 55.9 mm -> 28.4 x 56.2 mm
- board text added: "6.2018"
- board text added: "BOTTOM"
- board text added: "TOP"
- board text added: "v. 4"
- board text removed: "5.2018"
- board text removed: "Port 1, B: 2"
- board text removed: "Port 1, T: 1"
- board text removed: "Port 1, T: 3"
- board text removed: "Port 1, T: 4"
- board text removed: "v. 3"
